File: hardware/kicad/flowbench-main/field.kicad_sch (KiCad schematic)
At the start: 69 parts, among them J10 MAF (GX12-7), J11 Swirl encoder (GX12-5), J12 Bleed home switch (GX12-3), J13 Lift switches (GX12-4), J14 Orifice selector (GX12-5), J15 Motor current sensors (GX16-8), J16 Digimatic indicator (GX12-4), J17 UPDI, Q7 MMBT3904, Q8 MMBT3904, Q9 MMBT3904, U10 ATtiny1616-SN, U8 74LVC14 (5 V-tolerant inputs), U9 MCP6002

Commit message: KiCad: WIZ850io as one part with a two-row footprint
Pinout and size confirmed from the module (20 x 25 mm, two 1x6 headers).
The two header symbols become one 12-pin WIZ850io part on footprint
FlowBench:WIZ850io (J1 pads 1-6, J2 pads 7-12, rows 17.78 mm apart), so the
headers can't be placed at the wrong spacing.

Co-Authored-By: Claude Opus 5.5 <noreply@anthropic.com>
Claude-Session: https://claude.ai/code/session_01QEmmugJA9S77dSDSNcKrPa
Parts:
- removed J10: MAF (GX12-7), Connector_Phoenix_MC:PhoenixContact_MC_1,5_7-G-3.81_1x07_P3.81mm_Horizontal, symbol FlowBench:Conn_01x07
- removed J11: Swirl encoder (GX12-5), Connector_Phoenix_MC:PhoenixContact_MC_1,5_5-G-3.81_1x05_P3.81mm_Horizontal, symbol FlowBench:Conn_01x05
- removed J12: Bleed home switch (GX12-3), Connector_Phoenix_MC:PhoenixContact_MC_1,5_3-G-3.81_1x03_P3.81mm_Horizontal, symbol FlowBench:Conn_01x03
- removed J13: Lift switches (GX12-4), Connector_Phoenix_MC:PhoenixContact_MC_1,5_4-G-3.81_1x04_P3.81mm_Horizontal, symbol FlowBench:Conn_01x04
- removed J14: Orifice selector (GX12-5), Connector_Phoenix_MC:PhoenixContact_MC_1,5_5-G-3.81_1x05_P3.81mm_Horizontal, symbol FlowBench:Conn_01x05
- removed J15: Motor current sensors (GX16-8), Connector_Phoenix_MC:PhoenixContact_MC_1,5_8-G-3.81_1x08_P3.81mm_Horizontal, symbol FlowBench:Conn_01x08
- removed J16: Digimatic indicator (GX12-4), Connector_Phoenix_MC:PhoenixContact_MC_1,5_4-G-3.81_1x04_P3.81mm_Horizontal, symbol FlowBench:Conn_01x04
- removed J17: UPDI, Connector_PinHeader_2.54mm:PinHeader_1x03_P2.54mm_Vertical, symbol FlowBench:Conn_01x03
- removed U10: ATtiny1616-SN, Package_SO:SOIC-20W_7.5x12.8mm_P1.27mm, symbol FlowBench:ATtiny1616-S
- removed U8: 74LVC14 (5 V-tolerant inputs), Package_SO:SOIC-14_3.9x8.7mm_P1.27mm, symbol FlowBench:74LVC14
- removed U9: MCP6002, Package_SO:SOIC-8_3.9x4.9mm_P1.27mm, symbol FlowBench:MCP6002-xSN
- added J10: Bleed home switch (GX12-3), Connector_Phoenix_MC:PhoenixContact_MC_1,5_3-G-3.81_1x03_P3.81mm_Horizontal, symbol FlowBench:Conn_01x03
- added J11: Lift switches (GX12-4), Connector_Phoenix_MC:PhoenixContact_MC_1,5_4-G-3.81_1x04_P3.81mm_Horizontal, symbol FlowBench:Conn_01x04
- added J12: Orifice selector (GX12-5), Connector_Phoenix_MC:PhoenixContact_MC_1,5_5-G-3.81_1x05_P3.81mm_Horizontal, symbol FlowBench:Conn_01x05
- added J13: Motor current sensors (GX16-8), Connector_Phoenix_MC:PhoenixContact_MC_1,5_8-G-3.81_1x08_P3.81mm_Horizontal, symbol FlowBench:Conn_01x08
- added J14: Digimatic indicator (GX12-4), Connector_Phoenix_MC:PhoenixContact_MC_1,5_4-G-3.81_1x04_P3.81mm_Horizontal, symbol FlowBench:Conn_01x04
- added J15: UPDI, Connector_PinHeader_2.54mm:PinHeader_1x03_P2.54mm_Vertical, symbol FlowBench:Conn_01x03
- added J8: MAF (GX12-7), Connector_Phoenix_MC:PhoenixContact_MC_1,5_7-G-3.81_1x07_P3.81mm_Horizontal, symbol FlowBench:Conn_01x07
- added J9: Swirl encoder (GX12-5), Connector_Phoenix_MC:PhoenixContact_MC_1,5_5-G-3.81_1x05_P3.81mm_Horizontal, symbol FlowBench:Conn_01x05
- added U10: MCP6002, Package_SO:SOIC-8_3.9x4.9mm_P1.27mm, symbol FlowBench:MCP6002-xSN
- added U11: ATtiny1616-SN, Package_SO:SOIC-20W_7.5x12.8mm_P1.27mm, symbol FlowBench:ATtiny1616-S
- added U9: 74LVC14 (5 V-tolerant inputs), Package_SO:SOIC-14_3.9x8.7mm_P1.27mm, symbol FlowBench:74LVC14
Connections:
- net +24V_FIELD: now also J10.1 (Pin_1), J11.1 (Pin_1), J12.1 (Pin_1)
- net +3V3: now also J15.2 (Pin_2), U10.8 (V+), U11.1 (VCC), U9.14 (VCC)
- net +5V: now also J9.1 (Pin_1)
- net BLEED_HOME_IN: now also J10.2 (Pin_2)
- net CT1_IN: now also J13.1 (Pin_1)
- net CT2_IN: now also J13.2 (Pin_2)
- net CT3_IN: now also J13.3 (Pin_3)
- net CT4_IN: now also J13.4 (Pin_4)
- net CT5_IN: now also J13.5 (Pin_5)
- net CT6_IN: now also J13.6 (Pin_6)
- net CT_BIAS: now also J13.7 (Pin_7), U10.1, U10.2 (-)
- net CT_BIAS_DIV: now also U10.3 (+)
- net DIGI_CLK: now also J14.3 (Pin_3)
- net DIGI_CLK_MCU: now also U11.2 (PA4)
- net DIGI_DATA: now also J14.2 (Pin_2)
- net DIGI_DATA_MCU: now also U11.3 (PA5)
- net DIGI_REQ: now also J14.4 (Pin_4)
- net DIGI_REQ_DRV: now also U11.4 (PA6)
- net DIGI_UPDI: now also J15.1 (Pin_1), U11.16 (~{RESET}/PA0)
- net GND: now also J10.3 (Pin_3), J11.4 (Pin_4), J12.5 (Pin_5), J13.8 (Pin_8), J14.1 (Pin_1), J15.3 (Pin_3), J8.2 (Pin_2), J9.2 (Pin_2), U10.4 (V-), U10.5 (+), U11.20 (GND), U9.11, U9.13, U9.7 (GND), U9.9
- net LIFT_HOME_IN: now also J11.2 (Pin_2)
- net LIFT_MAX_IN: now also J11.3 (Pin_3)
- net MAF_12V: now also J8.1 (Pin_1)
- net MAF_5VREF: now also J8.6 (Pin_6)
- net MAF_FREQ: now also U9.2
- net MAF_FREQ_IN: now also J8.4 (Pin_4)
- net MAF_FREQ_P: now also U9.1
- net MAF_IAT: now also J8.5 (Pin_5)
- net MAF_ID: now also J8.7 (Pin_7)
- net MAF_SIG: now also J8.3 (Pin_3)
- net OPB_FB: now also U10.6 (-), U10.7
- net ORIF_B0_IN: now also J12.2 (Pin_2)
- net ORIF_B1_IN: now also J12.3 (Pin_3)
- net ORIF_B2_IN: now also J12.4 (Pin_4)
- net SCL: now also U11.11 (PB0)
- net SDA: now also U11.10 (PB1)
- net SWIRL_A: now also U9.4
- net SWIRL_A_IN: now also J9.3 (Pin_3)
- net SWIRL_A_P: now also U9.3
- net SWIRL_B: now also U9.6
- net SWIRL_B_IN: now also J9.4 (Pin_4)
- net SWIRL_B_P: now also U9.5

Commit message: KiCad: DevKit as one part with a 25.4 mm two-row footprint
Header pinout confirmed against Espressif's J1/J3 tables; row spacing measured
at 25.4 mm. The two header symbols become one 44-pin ESP32-S3-DevKitC-1 part on
footprint FlowBench:ESP32-S3-DevKitC-1 (J1 pads 1-22, J3 pads 23-44), with the
antenna end marked. BOM notes the N32R16V as a drop-in alternative.

Co-Authored-By: Claude Opus 5.5 <noreply@anthropic.com>
Claude-Session: https://claude.ai/code/session_01QEmmugJA9S77dSDSNcKrPa
Parts:
- removed J10: Bleed home switch (GX12-3), Connector_Phoenix_MC:PhoenixContact_MC_1,5_3-G-3.81_1x03_P3.81mm_Horizontal, symbol FlowBench:Conn_01x03
- removed J11: Lift switches (GX12-4), Connector_Phoenix_MC:PhoenixContact_MC_1,5_4-G-3.81_1x04_P3.81mm_Horizontal, symbol FlowBench:Conn_01x04
- removed J12: Orifice selector (GX12-5), Connector_Phoenix_MC:PhoenixContact_MC_1,5_5-G-3.81_1x05_P3.81mm_Horizontal, symbol FlowBench:Conn_01x05
- removed J13: Motor current sensors (GX16-8), Connector_Phoenix_MC:PhoenixContact_MC_1,5_8-G-3.81_1x08_P3.81mm_Horizontal, symbol FlowBench:Conn_01x08
- removed J14: Digimatic indicator (GX12-4), Connector_Phoenix_MC:PhoenixContact_MC_1,5_4-G-3.81_1x04_P3.81mm_Horizontal, symbol FlowBench:Conn_01x04
- removed J15: UPDI, Connector_PinHeader_2.54mm:PinHeader_1x03_P2.54mm_Vertical, symbol FlowBench:Conn_01x03
- removed J8: MAF (GX12-7), Connector_Phoenix_MC:PhoenixContact_MC_1,5_7-G-3.81_1x07_P3.81mm_Horizontal, symbol FlowBench:Conn_01x07
- removed J9: Swirl encoder (GX12-5), Connector_Phoenix_MC:PhoenixContact_MC_1,5_5-G-3.81_1x05_P3.81mm_Horizontal, symbol FlowBench:Conn_01x05
- removed U10: MCP6002, Package_SO:SOIC-8_3.9x4.9mm_P1.27mm, symbol FlowBench:MCP6002-xSN
- removed U11: ATtiny1616-SN, Package_SO:SOIC-20W_7.5x12.8mm_P1.27mm, symbol FlowBench:ATtiny1616-S
- removed U9: 74LVC14 (5 V-tolerant inputs), Package_SO:SOIC-14_3.9x8.7mm_P1.27mm, symbol FlowBench:74LVC14
- added J10: Orifice selector (GX12-5), Connector_Phoenix_MC:PhoenixContact_MC_1,5_5-G-3.81_1x05_P3.81mm_Horizontal, symbol FlowBench:Conn_01x05
- added J11: Motor current sensors (GX16-8), Connector_Phoenix_MC:PhoenixContact_MC_1,5_8-G-3.81_1x08_P3.81mm_Horizontal, symbol FlowBench:Conn_01x08
- added J12: Digimatic indicator (GX12-4), Connector_Phoenix_MC:PhoenixContact_MC_1,5_4-G-3.81_1x04_P3.81mm_Horizontal, symbol FlowBench:Conn_01x04
- added J13: UPDI, Connector_PinHeader_2.54mm:PinHeader_1x03_P2.54mm_Vertical, symbol FlowBench:Conn_01x03
- added J6: MAF (GX12-7), Connector_Phoenix_MC:PhoenixContact_MC_1,5_7-G-3.81_1x07_P3.81mm_Horizontal, symbol FlowBench:Conn_01x07
- added J7: Swirl encoder (GX12-5), Connector_Phoenix_MC:PhoenixContact_MC_1,5_5-G-3.81_1x05_P3.81mm_Horizontal, symbol FlowBench:Conn_01x05
- added J8: Bleed home switch (GX12-3), Connector_Phoenix_MC:PhoenixContact_MC_1,5_3-G-3.81_1x03_P3.81mm_Horizontal, symbol FlowBench:Conn_01x03
- added J9: Lift switches (GX12-4), Connector_Phoenix_MC:PhoenixContact_MC_1,5_4-G-3.81_1x04_P3.81mm_Horizontal, symbol FlowBench:Conn_01x04
- added U10: 74LVC14 (5 V-tolerant inputs), Package_SO:SOIC-14_3.9x8.7mm_P1.27mm, symbol FlowBench:74LVC14
- added U11: MCP6002, Package_SO:SOIC-8_3.9x4.9mm_P1.27mm, symbol FlowBench:MCP6002-xSN
- added U12: ATtiny1616-SN, Package_SO:SOIC-20W_7.5x12.8mm_P1.27mm, symbol FlowBench:ATtiny1616-S
Connections:
- net +24V_FIELD: now also J10.1 (Pin_1), J8.1 (Pin_1), J9.1 (Pin_1)
- net +3V3: now also J13.2 (Pin_2), U10.14 (VCC), U11.8 (V+), U12.1 (VCC)
- net +5V: now also J7.1 (Pin_1)
- net BLEED_HOME_IN: now also J8.2 (Pin_2)
- net CT1_IN: now also J11.1 (Pin_1)
- net CT2_IN: now also J11.2 (Pin_2)
- net CT3_IN: now also J11.3 (Pin_3)
- net CT4_IN: now also J11.4 (Pin_4)
- net CT5_IN: now also J11.5 (Pin_5)
- net CT6_IN: now also J11.6 (Pin_6)
- net CT_BIAS: now also J11.7 (Pin_7), U11.1, U11.2 (-)
- net CT_BIAS_DIV: now also U11.3 (+)
- net DIGI_CLK: now also J12.3 (Pin_3)
- net DIGI_CLK_MCU: now also U12.2 (PA4)
- net DIGI_DATA: now also J12.2 (Pin_2)
- net DIGI_DATA_MCU: now also U12.3 (PA5)
- net DIGI_REQ: now also J12.4 (Pin_4)
- net DIGI_REQ_DRV: now also U12.4 (PA6)
- net DIGI_UPDI: now also J13.1 (Pin_1), U12.16 (~{RESET}/PA0)
- net GND: now also J10.5 (Pin_5), J11.8 (Pin_8), J12.1 (Pin_1), J13.3 (Pin_3), J6.2 (Pin_2), J7.2 (Pin_2), J8.3 (Pin_3), J9.4 (Pin_4), U10.11, U10.13, U10.7 (GND), U10.9, U11.4 (V-), U11.5 (+), U12.20 (GND)
- net LIFT_HOME_IN: now also J9.2 (Pin_2)
- net LIFT_MAX_IN: now also J9.3 (Pin_3)
- net MAF_12V: now also J6.1 (Pin_1)
- net MAF_5VREF: now also J6.6 (Pin_6)
- net MAF_FREQ: now also U10.2
- net MAF_FREQ_IN: now also J6.4 (Pin_4)
- net MAF_FREQ_P: now also U10.1
- net MAF_IAT: now also J6.5 (Pin_5)
- net MAF_ID: now also J6.7 (Pin_7)
- net MAF_SIG: now also J6.3 (Pin_3)
- net OPB_FB: now also U11.6 (-), U11.7
- net ORIF_B0_IN: now also J10.2 (Pin_2)
- net ORIF_B1_IN: now also J10.3 (Pin_3)
- net ORIF_B2_IN: now also J10.4 (Pin_4)
- net SCL: now also U12.11 (PB0)
- net SDA: now also U12.10 (PB1)
- net SWIRL_A: now also U10.4
- net SWIRL_A_IN: now also J7.3 (Pin_3)
- net SWIRL_A_P: now also U10.3
- net SWIRL_B: now also U10.6
- net SWIRL_B_IN: now also J7.4 (Pin_4)
- net SWIRL_B_P: now also U10.5
