File: hardware/kicad/flowbench-main/field.kicad_sch (KiCad schematic)
At the start: 69 parts, among them J10 Orifice selector (GX12-5), J11 Motor current sensors (GX16-8), J12 Digimatic indicator (GX12-4), J13 UPDI, J6 MAF (GX12-7), J7 Swirl encoder (GX12-5), J8 Bleed home switch (GX12-3), J9 Lift switches (GX12-4), Q7 MMBT3904, Q8 MMBT3904, Q9 MMBT3904, U10 74LVC14 (5 V-tolerant inputs), U11 MCP6002, U12 ATtiny1616-SN

Commit message: KiCad: 180 x 125 mm layout, status LEDs, grouped test-point areas
- Board shrinks from 220 x 160 to 180 x 125 mm with connectors on all four
  edges; 1.0 mm between parts kept for hand soldering.
- 24 status LEDs: power rails, eFuse fault, stepper alarms, watchdog, armed,
  stepper power, each contactor coil, and every switch input (in series with
  its opto, no extra resistor).
- Scattered test points replaced by grouped areas: 24 V loops, logic-supply
  loops, and controller, analog and Digimatic 2-row headers with a GND row.
  No test points on SPI/SD lines.
- LED, test point and test header labels stay on the silkscreen.

Co-Authored-By: Claude Opus 5.5 <noreply@anthropic.com>
Claude-Session: https://claude.ai/code/session_01QEmmugJA9S77dSDSNcKrPa
Parts:
- removed J6: MAF (GX12-7), Connector_Phoenix_MC:PhoenixContact_MC_1,5_7-G-3.81_1x07_P3.81mm_Horizontal, symbol FlowBench:Conn_01x07
- removed J7: Swirl encoder (GX12-5), Connector_Phoenix_MC:PhoenixContact_MC_1,5_5-G-3.81_1x05_P3.81mm_Horizontal, symbol FlowBench:Conn_01x05
- removed R42: 100R, Resistor_SMD:R_0805_2012Metric, symbol FlowBench:R
- removed R43, R47: 1k, Resistor_SMD:R_0805_2012Metric, symbol FlowBench:R
- removed R44: 15k, Resistor_SMD:R_0805_2012Metric, symbol FlowBench:R
- removed R45, R48: 10k, Resistor_SMD:R_0805_2012Metric, symbol FlowBench:R
- removed R46: 2.49k, Resistor_SMD:R_0805_2012Metric, symbol FlowBench:R
- removed TP19: DIGI_CLK, TestPoint:TestPoint_Loop_D2.50mm_Drill1.0mm, symbol FlowBench:TestPoint
- removed TP20: DIGI_DATA, TestPoint:TestPoint_Loop_D2.50mm_Drill1.0mm, symbol FlowBench:TestPoint
- removed TP21: DIGI_REQ, TestPoint:TestPoint_Loop_D2.50mm_Drill1.0mm, symbol FlowBench:TestPoint
- added J14: Digimatic indicator (GX12-4), Connector_Phoenix_MC:PhoenixContact_MC_1,5_4-G-3.81_1x04_P3.81mm_Horizontal, symbol FlowBench:Conn_01x04
- added J15: UPDI, Connector_PinHeader_2.54mm:PinHeader_1x03_P2.54mm_Vertical, symbol FlowBench:Conn_01x03
- added J16: Digimatic test header, Connector_PinHeader_2.54mm:PinHeader_2x03_P2.54mm_Vertical, symbol FlowBench:Conn_02x03_Odd_Even
- added R73, R74, R75, R76, R77, R78: 10k, Resistor_SMD:R_0805_2012Metric, symbol FlowBench:R
- added R79: 100k, Resistor_SMD:R_0805_2012Metric, symbol FlowBench:R
- J10: value Orifice selector (GX12-5) -> Bleed home switch (GX12-3); footprint Connector_Phoenix_MC:PhoenixContact_MC_1,5_5-G-3.81_1x05_P3.81mm_Horizontal -> Connector_Phoenix_MC:PhoenixContact_MC_1,5_3-G-3.81_1x03_P3.81mm_Horizontal; symbol FlowBench:Conn_01x05 -> FlowBench:Conn_01x03
- J11: value Motor current sensors (GX16-8) -> Lift switches (GX12-4); footprint Connector_Phoenix_MC:PhoenixContact_MC_1,5_8-G-3.81_1x08_P3.81mm_Horizontal -> Connector_Phoenix_MC:PhoenixContact_MC_1,5_4-G-3.81_1x04_P3.81mm_Horizontal; symbol FlowBench:Conn_01x08 -> FlowBench:Conn_01x04
- J12: value Digimatic indicator (GX12-4) -> Orifice selector (GX12-5); footprint Connector_Phoenix_MC:PhoenixContact_MC_1,5_4-G-3.81_1x04_P3.81mm_Horizontal -> Connector_Phoenix_MC:PhoenixContact_MC_1,5_5-G-3.81_1x05_P3.81mm_Horizontal; symbol FlowBench:Conn_01x04 -> FlowBench:Conn_01x05
- J13: value UPDI -> Motor current sensors (GX16-8); footprint Connector_PinHeader_2.54mm:PinHeader_1x03_P2.54mm_Vertical -> Connector_Phoenix_MC:PhoenixContact_MC_1,5_8-G-3.81_1x08_P3.81mm_Horizontal; symbol FlowBench:Conn_01x03 -> FlowBench:Conn_01x08
- J8: value Bleed home switch (GX12-3) -> MAF (GX12-7); footprint Connector_Phoenix_MC:PhoenixContact_MC_1,5_3-G-3.81_1x03_P3.81mm_Horizontal -> Connector_Phoenix_MC:PhoenixContact_MC_1,5_7-G-3.81_1x07_P3.81mm_Horizontal; symbol FlowBench:Conn_01x03 -> FlowBench:Conn_01x07
- J9: value Lift switches (GX12-4) -> Swirl encoder (GX12-5); footprint Connector_Phoenix_MC:PhoenixContact_MC_1,5_4-G-3.81_1x04_P3.81mm_Horizontal -> Connector_Phoenix_MC:PhoenixContact_MC_1,5_5-G-3.81_1x05_P3.81mm_Horizontal; symbol FlowBench:Conn_01x04 -> FlowBench:Conn_01x05
- R49: value 1k -> 100R
- R50: value 4.7k -> 1k
- R51: value 1k -> 15k
- R53: value 4.7k -> 2.49k
- R55: value 4.7k -> 10k
- R57: value 10k -> 4.7k
- R58, R66, R67, R68, R69, R70, R71: value 10k -> 1k
- R59, R64: value 1k -> 10k
- R60, R62: value 1k -> 4.7k
- R72: value 100k -> 10k
Connections:
- net +24V_FIELD: now also J11.1 (Pin_1), J12.1 (Pin_1); no longer J8.1 (Pin_1), J9.1 (Pin_1)
- net +3V3: now also R64.1, R72.1, J15.2 (Pin_2), R74.1, R75.1, R77.1; no longer J13.2 (Pin_2), R57.1, R65.1, R67.1, R68.1, R70.1
- net +5V: now also J9.1 (Pin_1), R57.2, R60.1, R62.1; no longer R50.2, R53.1, R55.1
- net +5VA: now also R49.1, R53.1, R55.1
- net BLEED_HOME_IN: now also J10.2 (Pin_2); no longer J8.2 (Pin_2)
- net CT1: now also R66.2; no longer R59.2
- net CT1_IN: now also J13.1 (Pin_1), R66.1; no longer J11.1 (Pin_1), R59.1
- net CT2: now also R67.2; no longer R60.2
- net CT2_IN: now also J13.2 (Pin_2), R67.1; no longer J11.2 (Pin_2), R60.1
- net CT3: now also R68.2; no longer R61.2
- net CT3_IN: now also J13.3 (Pin_3), R68.1; no longer J11.3 (Pin_3), R61.1
- net CT4: now also R69.2; no longer R62.2
- net CT4_IN: now also J13.4 (Pin_4), R69.1; no longer J11.4 (Pin_4), R62.1
- net CT5: now also R70.2; no longer R63.2
- net CT5_IN: now also J13.5 (Pin_5), R70.1; no longer J11.5 (Pin_5), R63.1
- net CT6: now also R71.2; no longer R64.2
- net CT6_IN: now also J13.6 (Pin_6), R71.1; no longer J11.6 (Pin_6), R64.1
- net CT_BIAS: now also J13.7 (Pin_7); no longer J11.7 (Pin_7)
- net CT_BIAS_DIV: now also R64.2, R65.1; no longer R57.2, R58.1
- net DIGI_CLK: now also R72.2, J14.3 (Pin_3), J16.1 (Pin_1), R73.1; no longer J12.3 (Pin_3), R65.2, R66.1
- net DIGI_CLK_INV: now also R74.2; no longer R67.2
- net DIGI_CLK_QB: now also R73.2; no longer R66.2
- net DIGI_DATA: now also J14.2 (Pin_2), J16.3 (Pin_3), R75.2, R76.1; no longer J12.2 (Pin_2), R68.2, R69.1
- net DIGI_DATA_INV: now also R77.2; no longer R70.2
- net DIGI_DATA_QB: now also R76.2; no longer R69.2
- net DIGI_REQ: now also J14.4 (Pin_4), J16.5 (Pin_5); no longer J12.4 (Pin_4)
- net DIGI_REQ_B: now also R78.2, R79.1; no longer R71.2, R72.1
- net DIGI_REQ_DRV: now also R78.1; no longer R71.1
- net DIGI_UPDI: now also J15.1 (Pin_1); no longer J13.1 (Pin_1)
- net GND: now also J10.3 (Pin_3), J11.4 (Pin_4), J12.5 (Pin_5), J13.8 (Pin_8), J8.2 (Pin_2), J9.2 (Pin_2), R59.2, R65.2, J14.1 (Pin_1), J15.3 (Pin_3), J16.2 (Pin_2), J16.4 (Pin_4), J16.6 (Pin_6), R79.2; no longer J10.5 (Pin_5), J11.8 (Pin_8), J12.1 (Pin_1), J13.3 (Pin_3), J8.3 (Pin_3), J9.4 (Pin_4), R58.2, R72.2
- net LIFT_HOME_IN: now also J11.2 (Pin_2); no longer J9.2 (Pin_2)
- net LIFT_MAX_IN: now also J11.3 (Pin_3); no longer J9.3 (Pin_3)
- net MAF_12V: now also J8.1 (Pin_1)
- net MAF_5VREF: now also J8.6 (Pin_6), R49.2
- net MAF_FREQ_IN: now also J8.4 (Pin_4), R58.1; no longer R51.1
- net MAF_FREQ_P: now also R58.2, R59.1; no longer R51.2, R52.1
- net MAF_FREQ_PU: now also R57.1; no longer R50.1
- net MAF_IAT: now also J8.5 (Pin_5), R53.2, R54.1
- net MAF_IAT_ADC: now also R54.2
- net MAF_ID: now also J8.7 (Pin_7), R55.2, R56.1; no longer R49.1
- net MAF_ID_ADC: now also R56.2; no longer R49.2
- net MAF_SIG: now also J8.3 (Pin_3), R50.1
- net MAF_SIG_ADC: now also R51.2, R52.1
- net MAF_SIG_P: now also R50.2, R51.1
- net ORIF_B0_IN: now also J12.2 (Pin_2); no longer J10.2 (Pin_2)
- net ORIF_B1_IN: now also J12.3 (Pin_3); no longer J10.3 (Pin_3)
- net ORIF_B2_IN: now also J12.4 (Pin_4); no longer J10.4 (Pin_4)
- net SWIRL_A_IN: now also J9.3 (Pin_3), R60.2, R61.1; no longer R53.2, R54.1
- net SWIRL_A_P: now also R61.2; no longer R54.2
- net SWIRL_B_IN: now also J9.4 (Pin_4), R62.2, R63.1; no longer R55.2, R56.1
- net SWIRL_B_P: now also R63.2; no longer R56.2
Other:
- moved on the sheet: R49, R50, R51, R52, R53, R54, R55, R56, R57, R58, R59, R60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

Commit message: KiCad: prototyping area with I2C expansion header
- 10 x 7 plated-hole grid (+3V3 row, +5V row, 4 free rows, GND row) between
  the optocouplers and the multiplexer; footprint FlowBench:ProtoArea_10x7.
- Multiplexer channels 4-7 now brought out with 4.7k pull-ups to a new I2C
  expansion header beside the grid; the expander 2 spare header moves there too.
- ATtiny, 74LVC14 and Digimatic test header nudged to keep 1 mm clearance.

Co-Authored-By: Claude Opus 5.5 <noreply@anthropic.com>
Claude-Session: https://claude.ai/code/session_01QEmmugJA9S77dSDSNcKrPa
Parts:
- removed R49: 100R, Resistor_SMD:R_0805_2012Metric, symbol FlowBench:R
- removed R50, R54, R56: 1k, Resistor_SMD:R_0805_2012Metric, symbol FlowBench:R
- removed R51: 15k, Resistor_SMD:R_0805_2012Metric, symbol FlowBench:R
- removed R52, R55: 10k, Resistor_SMD:R_0805_2012Metric, symbol FlowBench:R
- removed R53: 2.49k, Resistor_SMD:R_0805_2012Metric, symbol FlowBench:R
- added R80, R81, R82, R83, R84, R85, R86: 10k, Resistor_SMD:R_0805_2012Metric, symbol FlowBench:R
- added R87: 100k, Resistor_SMD:R_0805_2012Metric, symbol FlowBench:R
- R57: value 4.7k -> 100R
- R59: value 10k -> 15k
- R60: value 4.7k -> 10k
- R61: value 1k -> 2.49k
- R62: value 4.7k -> 1k
- R63, R67: value 1k -> 10k
- R64, R74, R75, R76, R77, R78: value 10k -> 1k
- R65: value 10k -> 4.7k
- R68, R70: value 1k -> 4.7k
- R79: value 100k -> 1k
Connections:
- net +3V3: now also R80.1, R82.1, R83.1, R85.1; no longer R64.1, R74.1, R75.1, R77.1
- net +5V: now also R65.2, R68.1, R70.1; no longer R57.2, R60.1, R62.1
- net +5VA: now also R57.1, R61.1, R63.1
- net CT1: now also R74.2; no longer R66.2
- net CT1_IN: now also R74.1; no longer R66.1
- net CT2: now also R75.2; no longer R67.2
- net CT2_IN: now also R75.1; no longer R67.1
- net CT3: now also R76.2; no longer R68.2
- net CT3_IN: now also R76.1; no longer R68.1
- net CT4: now also R77.2; no longer R69.2
- net CT4_IN: now also R77.1; no longer R69.1
- net CT5: now also R78.2; no longer R70.2
- net CT5_IN: now also R78.1; no longer R70.1
- net CT6: now also R79.2; no longer R71.2
- net CT6_IN: now also R79.1; no longer R71.1
- net CT_BIAS_DIV: now also R72.2, R73.1; no longer R64.2, R65.1
- net DIGI_CLK: now also R80.2, R81.1; no longer R72.2, R73.1
- net DIGI_CLK_INV: now also R82.2; no longer R74.2
- net DIGI_CLK_QB: now also R81.2; no longer R73.2
- net DIGI_DATA: now also R83.2, R84.1; no longer R75.2, R76.1
- net DIGI_DATA_INV: now also R85.2; no longer R77.2
- net DIGI_DATA_QB: now also R84.2; no longer R76.2
- net DIGI_REQ_B: now also R86.2, R87.1; no longer R78.2, R79.1
- net DIGI_REQ_DRV: now also R86.1; no longer R78.1
- net GND: now also R60.2, R67.2, R73.2, R87.2; no longer R59.2, R65.2, R79.2
- net MAF_5VREF: now also R57.2
- net MAF_FREQ_IN: now also R66.1; no longer R58.1
- net MAF_FREQ_P: now also R66.2, R67.1; no longer R58.2, R59.1
- net MAF_FREQ_PU: now also R65.1; no longer R57.1
- net MAF_IAT: now also R61.2, R62.1
- net MAF_IAT_ADC: now also R62.2
- net MAF_ID: now also R63.2, R64.1
- net MAF_ID_ADC: now also R64.2
- net MAF_SIG: now also R58.1
- net MAF_SIG_ADC: now also R59.2, R60.1
- net MAF_SIG_P: now also R58.2, R59.1
- net SWIRL_A_IN: now also R68.2, R69.1; no longer R60.2, R61.1
- net SWIRL_A_P: now also R69.2; no longer R61.2
- net SWIRL_B_IN: now also R70.2, R71.1; no longer R62.2, R63.1
- net SWIRL_B_P: now also R71.2; no longer R63.2
Other:
- moved on the sheet: R57, R58, R59, R60, R61, R62, R63, R64, R65, R66, R67, R68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
