File: hardware/kicad/flowbench-main/io.kicad_sch (KiCad schematic)
At the start: 57 parts, among them J14 Expander 2 spare, J15 Bleed stepper signals (GX16-8), J16 Bleed stepper 24 V (GX12-2), J17 Lift stepper signals (GX16-8), J18 Lift stepper 24 V (GX12-2), J19 Motor housing coils (GX16-8), J20 Motors-armed lamp, J21 E-stop (2 NC contacts), U13 TCA9535PWR #1 (0x20), U14 TCA9535PWR #2 (0x21), U15 TLP291-4, U16 TLP291-4, U17 TLP291-4, U18 AM26C31 (bleed stepper), U19 AM26C31 (lift stepper), U20 TBD62083AFWG, U21 74HCT123

Commit message: KiCad: 180 x 125 mm layout, status LEDs, grouped test-point areas
- Board shrinks from 220 x 160 to 180 x 125 mm with connectors on all four
  edges; 1.0 mm between parts kept for hand soldering.
- 24 status LEDs: power rails, eFuse fault, stepper alarms, watchdog, armed,
  stepper power, each contactor coil, and every switch input (in series with
  its opto, no extra resistor).
- Scattered test points replaced by grouped areas: 24 V loops, logic-supply
  loops, and controller, analog and Digimatic 2-row headers with a GND row.
  No test points on SPI/SD lines.
- LED, test point and test header labels stay on the silkscreen.

Co-Authored-By: Claude Opus 5.5 <noreply@anthropic.com>
Claude-Session: https://claude.ai/code/session_01QEmmugJA9S77dSDSNcKrPa
Parts:
- removed J14: Expander 2 spare, Connector_PinHeader_2.54mm:PinHeader_1x10_P2.54mm_Vertical, symbol FlowBench:Conn_01x10
- removed J15: Bleed stepper signals (GX16-8), Connector_Phoenix_MC:PhoenixContact_MC_1,5_8-G-3.81_1x08_P3.81mm_Horizontal, symbol FlowBench:Conn_01x08
- removed J16: Bleed stepper 24 V (GX12-2), Connector_Phoenix_MSTB:PhoenixContact_MSTBA_2,5_2-G-5,08_1x02_P5.08mm_Horizontal, symbol FlowBench:Conn_01x02
- removed R73, R74, R75, R76, R77, R78, R79: 10k, Resistor_SMD:R_0805_2012Metric, symbol FlowBench:R
- removed TP22: WD_OK, TestPoint:TestPoint_Loop_D2.50mm_Drill1.0mm, symbol FlowBench:TestPoint
- added J22: Motor housing coils (GX16-8), Connector_Phoenix_MC:PhoenixContact_MC_1,5_8-G-3.81_1x08_P3.81mm_Horizontal, symbol FlowBench:Conn_01x08
- added J23: Motors-armed lamp, Connector_Phoenix_MC:PhoenixContact_MC_1,5_2-G-3.81_1x02_P3.81mm_Horizontal, symbol FlowBench:Conn_01x02
- added J24: E-stop (2 NC contacts), Connector_Phoenix_MC:PhoenixContact_MC_1,5_4-G-3.81_1x04_P3.81mm_Horizontal, symbol FlowBench:Conn_01x04
- added LED10: LIFT HOME, LED_SMD:LED_0805_2012Metric, symbol FlowBench:LED
- added LED11: LIFT MAX, LED_SMD:LED_0805_2012Metric, symbol FlowBench:LED
- added LED12: ORIF 0, LED_SMD:LED_0805_2012Metric, symbol FlowBench:LED
- added LED13: ORIF 1, LED_SMD:LED_0805_2012Metric, symbol FlowBench:LED
- added LED14: ORIF 2, LED_SMD:LED_0805_2012Metric, symbol FlowBench:LED
- added LED15: BLEED ALM, LED_SMD:LED_0805_2012Metric, symbol FlowBench:LED
- added LED16: LIFT ALM, LED_SMD:LED_0805_2012Metric, symbol FlowBench:LED
- added LED17: WD OK, LED_SMD:LED_0805_2012Metric, symbol FlowBench:LED
- added LED18: ARMED, LED_SMD:LED_0805_2012Metric, symbol FlowBench:LED
- added LED19: K1, LED_SMD:LED_0805_2012Metric, symbol FlowBench:LED
- added LED20: K2, LED_SMD:LED_0805_2012Metric, symbol FlowBench:LED
- added LED21: K3, LED_SMD:LED_0805_2012Metric, symbol FlowBench:LED
- added LED22: K4, LED_SMD:LED_0805_2012Metric, symbol FlowBench:LED
- added LED23: K5, LED_SMD:LED_0805_2012Metric, symbol FlowBench:LED
- added LED24: K6, LED_SMD:LED_0805_2012Metric, symbol FlowBench:LED
- added LED8: ESTOP OK, LED_SMD:LED_0805_2012Metric, symbol FlowBench:LED
- added LED9: BLEED HOME, LED_SMD:LED_0805_2012Metric, symbol FlowBench:LED
- added R106, R107, R108, R109: 4.7k, Resistor_SMD:R_0805_2012Metric, symbol FlowBench:R
- added R110, R111: 470R, Resistor_SMD:R_0805_2012Metric, symbol FlowBench:R
- added R112: 220k, Resistor_SMD:R_0805_2012Metric, symbol FlowBench:R
- added R113: 1.5k, Resistor_SMD:R_0805_2012Metric, symbol FlowBench:R
- added R114, R115, R116, R117, R118, R119, R120: 10k, Resistor_SMD:R_0805_2012Metric, symbol FlowBench:R
- J17: value Lift stepper signals (GX16-8) -> Expander 2 spare; footprint Connector_Phoenix_MC:PhoenixContact_MC_1,5_8-G-3.81_1x08_P3.81mm_Horizontal -> Connector_PinHeader_2.54mm:PinHeader_1x10_P2.54mm_Vertical; symbol FlowBench:Conn_01x08 -> FlowBench:Conn_01x10
- J18: value Lift stepper 24 V (GX12-2) -> Bleed stepper signals (GX16-8); footprint Connector_Phoenix_MSTB:PhoenixContact_MSTBA_2,5_2-G-5,08_1x02_P5.08mm_Horizontal -> Connector_Phoenix_MC:PhoenixContact_MC_1,5_8-G-3.81_1x08_P3.81mm_Horizontal; symbol FlowBench:Conn_01x02 -> FlowBench:Conn_01x08
- J19: value Motor housing coils (GX16-8) -> Bleed stepper 24 V (GX12-2); footprint Connector_Phoenix_MC:PhoenixContact_MC_1,5_8-G-3.81_1x08_P3.81mm_Horizontal -> Connector_Phoenix_MSTB:PhoenixContact_MSTBA_2,5_2-G-5,08_1x02_P5.08mm_Horizontal; symbol FlowBench:Conn_01x08 -> FlowBench:Conn_01x02
- J20: value Motors-armed lamp -> Lift stepper signals (GX16-8); footprint Connector_Phoenix_MC:PhoenixContact_MC_1,5_2-G-3.81_1x02_P3.81mm_Horizontal -> Connector_Phoenix_MC:PhoenixContact_MC_1,5_8-G-3.81_1x08_P3.81mm_Horizontal; symbol FlowBench:Conn_01x02 -> FlowBench:Conn_01x08
- J21: value E-stop (2 NC contacts) -> Lift stepper 24 V (GX12-2); footprint Connector_Phoenix_MC:PhoenixContact_MC_1,5_4-G-3.81_1x04_P3.81mm_Horizontal -> Connector_Phoenix_MSTB:PhoenixContact_MSTBA_2,5_2-G-5,08_1x02_P5.08mm_Horizontal; symbol FlowBench:Conn_01x04 -> FlowBench:Conn_01x02
- R100, R101, R102, R96, R97, R98, R99: value 4.7k -> 10k
- R103, R104: value 470R -> 4.7k
- R105: value 220k -> 4.7k
Connections:
- net +24V_FIELD: now also J24.3 (Pin_3); no longer J21.3 (Pin_3)
- net +3V3: now also J17.9 (Pin_9), R100.1, R101.1, R102.1, R80.1, R96.1, R97.1, R98.1, R99.1; no longer R85.1, R86.1, R87.1, R88.1, R89.1, R90.1, R91.1
- net +5V: now also R110.1, R111.1, R112.1; no longer R103.1, R104.1, R105.1
- net BLEED_24V_F: now also J19.1 (Pin_1)
- net BLEED_ALM_LED: now also LED15.1 (K); no longer R103.2
- net BLEED_ALM_N: now also R100.2; no longer R93.2
- net BLEED_ALM_P: now also J18.7 (Pin_7)
- net BLEED_DIR_N: now also J18.4 (Pin_4)
- net BLEED_DIR_P: now also J18.3 (Pin_3)
- net BLEED_ENA: now also R90.1; no longer R83.1
- net BLEED_ENA_N: now also J18.6 (Pin_6)
- net BLEED_ENA_P: now also J18.5 (Pin_5)
- net BLEED_HOME_IN: now also R104.1; no longer R97.1
- net BLEED_HOME_IN_LED: now also LED9.1 (K); no longer R97.2
- net BLEED_HOME_N: now also R93.2; no longer R86.2
- net BLEED_PUL_N: now also J18.2 (Pin_2)
- net BLEED_PUL_P: now also J18.1 (Pin_1)
- net BLEED_PWR_EN: now also R88.1; no longer R81.1
- net COIL1_CMD: now also R81.1
- net COIL1_RET: now also J22.2 (Pin_2), LED19.1 (K); no longer J19.2 (Pin_2)
- net COIL2_CMD: now also R82.1
- net COIL2_RET: now also J22.3 (Pin_3), LED20.1 (K); no longer J19.3 (Pin_3)
- net COIL3_CMD: now also R83.1
- net COIL3_RET: now also J22.4 (Pin_4), LED21.1 (K); no longer J19.4 (Pin_4)
- net COIL4_CMD: now also R84.1
- net COIL4_RET: now also J22.5 (Pin_5), LED22.1 (K); no longer J19.5 (Pin_5)
- net COIL5_CMD: now also R85.1
- net COIL5_RET: now also J22.6 (Pin_6), LED23.1 (K); no longer J19.6 (Pin_6)
- net COIL6_CMD: now also R86.1
- net COIL6_RET: now also J22.7 (Pin_7), LED24.1 (K); no longer J19.7 (Pin_7)
- net COIL_24V: now also J24.1 (Pin_1); no longer J21.1 (Pin_1)
- net COIL_24V_ESTOP: now also J22.1 (Pin_1), J23.1 (Pin_1), J24.2 (Pin_2), R114.1, R115.1, R116.1, R117.1, R118.1, R119.1, R120.1; no longer J19.1 (Pin_1), J20.1 (Pin_1), J21.2 (Pin_2)
- net EFUSE_FLT_N: now also R101.2; no longer R94.2
- net ESTOP_OK_N: now also R92.2; no longer R85.2
- net ESTOP_STAT_IN: now also R103.1, J24.4 (Pin_4); no longer J21.4 (Pin_4), R96.1
- net ESTOP_STAT_IN_LED: now also LED8.1 (K); no longer R96.2
- net ETH_INT_EXP: now also R102.2; no longer R95.2
- net EXP2_P10: now also J17.1 (Pin_1)
- net EXP2_P11: now also J17.2 (Pin_2)
- net EXP2_P12: now also J17.3 (Pin_3)
- net EXP2_P13: now also J17.4 (Pin_4)
- net EXP2_P14: now also J17.5 (Pin_5)
- net EXP2_P15: now also J17.6 (Pin_6)
- net EXP2_P16: now also J17.7 (Pin_7)
- net EXP2_P17: now also J17.8 (Pin_8)
- net EXP_INT_N: now also R80.2
- net GND: now also J17.10 (Pin_10), J18.8 (Pin_8), J19.2 (Pin_2), J20.8 (Pin_8), J21.2 (Pin_2), R85.2, R86.2, R87.2, R88.2, R89.2, R90.2, R91.2, LED17.1 (K), LED18.1 (K); no longer J17.8 (Pin_8), J18.2 (Pin_2), R80.2
- net LAMP_CMD: now also R87.1; no longer R80.1
- net LAMP_RET: now also J23.2 (Pin_2); no longer J20.2 (Pin_2)
- net LIFT_24V_F: now also J21.1 (Pin_1); no longer J18.1 (Pin_1)
- net LIFT_ALM_LED: now also LED16.1 (K); no longer R104.2
- net LIFT_ALM_N: now also R97.2; no longer R90.2
- net LIFT_ALM_P: now also J20.7 (Pin_7); no longer J17.7 (Pin_7)
- net LIFT_DIR_N: now also J20.4 (Pin_4); no longer J17.4 (Pin_4)
- net LIFT_DIR_P: now also J20.3 (Pin_3); no longer J17.3 (Pin_3)
- net LIFT_ENA: now also R91.1; no longer R84.1
- net LIFT_ENA_N: now also J20.6 (Pin_6); no longer J17.6 (Pin_6)
- net LIFT_ENA_P: now also J20.5 (Pin_5); no longer J17.5 (Pin_5)
- net LIFT_HOME_IN: now also R105.1; no longer R98.1
- net LIFT_HOME_IN_LED: now also LED10.1 (K); no longer R98.2
- net LIFT_HOME_N: now also R98.2; no longer R91.2
- net LIFT_MAX_IN: now also R106.1; no longer R99.1
- net LIFT_MAX_IN_LED: now also LED11.1 (K); no longer R99.2
- net LIFT_MAX_N: now also R99.2; no longer R92.2
- net LIFT_PUL_N: now also J20.2 (Pin_2); no longer J17.2 (Pin_2)
- net LIFT_PUL_P: now also J20.1 (Pin_1); no longer J17.1 (Pin_1)
- net LIFT_PWR_EN: now also R89.1; no longer R82.1
- net ORIF_B0_IN: now also R107.1; no longer R100.1
- net ORIF_B0_IN_LED: now also LED12.1 (K); no longer R100.2
- net ORIF_B0_N: now also R94.2; no longer R87.2
- net ORIF_B1_IN: now also R108.1; no longer R101.1
- net ORIF_B1_IN_LED: now also LED13.1 (K); no longer R101.2
- net ORIF_B1_N: now also R95.2; no longer R88.2
- net ORIF_B2_IN: now also R109.1; no longer R102.1
- net ORIF_B2_IN_LED: now also LED14.1 (K); no longer R102.2
- net ORIF_B2_N: now also R96.2; no longer R89.2
- net WD_OK: now also R113.1
- net WD_RC: now also R112.2; no longer R105.2
- new net BLEED_ALM_R: LED15.2 (A), R110.2
- new net BLEED_HOME_IN_R: LED9.2 (A), R104.2
- new net ESTOP_STAT_IN_R: LED8.2 (A), R103.2
- new net LED_ARMED_A: LED18.2 (A), R114.2
- new net LED_K1_A: LED19.2 (A), R115.2
- new net LED_K2_A: LED20.2 (A), R116.2
- new net LED_K3_A: LED21.2 (A), R117.2
- new net LED_K4_A: LED22.2 (A), R118.2
- new net LED_K5_A: LED23.2 (A), R119.2
- new net LED_K6_A: LED24.2 (A), R120.2
- new net LED_WD_A: LED17.2 (A), R113.2
- new net LIFT_ALM_R: LED16.2 (A), R111.2
- new net LIFT_HOME_IN_R: LED10.2 (A), R105.2
- new net LIFT_MAX_IN_R: LED11.2 (A), R106.2
- new net ORIF_B0_IN_R: LED12.2 (A), R107.2
- new net ORIF_B1_IN_R: LED13.2 (A), R108.2
- new net ORIF_B2_IN_R: LED14.2 (A), R109.2
Other:
- moved on the sheet: C38, C39, C40, C41, R100, R101, R102, R103, R104, R105, R80, R81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

Commit message: KiCad: prototyping area with I2C expansion header
- 10 x 7 plated-hole grid (+3V3 row, +5V row, 4 free rows, GND row) between
  the optocouplers and the multiplexer; footprint FlowBench:ProtoArea_10x7.
- Multiplexer channels 4-7 now brought out with 4.7k pull-ups to a new I2C
  expansion header beside the grid; the expander 2 spare header moves there too.
- ATtiny, 74LVC14 and Digimatic test header nudged to keep 1 mm clearance.

Co-Authored-By: Claude Opus 5.5 <noreply@anthropic.com>
Claude-Session: https://claude.ai/code/session_01QEmmugJA9S77dSDSNcKrPa
Parts:
- removed R80, R81, R82, R83, R84, R85, R86, R87: 10k, Resistor_SMD:R_0805_2012Metric, symbol FlowBench:R
- added J25: E-stop (2 NC contacts), Connector_Phoenix_MC:PhoenixContact_MC_1,5_4-G-3.81_1x04_P3.81mm_Horizontal, symbol FlowBench:Conn_01x04
- added PROTO1: Prototyping area, FlowBench:ProtoArea_10x7, symbol FlowBench:ProtoArea
- added R121: 1.5k, Resistor_SMD:R_0805_2012Metric, symbol FlowBench:R
- added R122, R123, R124, R125, R126, R127, R128: 10k, Resistor_SMD:R_0805_2012Metric, symbol FlowBench:R
- J18: value Bleed stepper signals (GX16-8) -> I2C expansion (mux ch4-7); footprint Connector_Phoenix_MC:PhoenixContact_MC_1,5_8-G-3.81_1x08_P3.81mm_Horizontal -> Connector_PinHeader_2.54mm:PinHeader_1x10_P2.54mm_Vertical; symbol FlowBench:Conn_01x08 -> FlowBench:Conn_01x10
- J19: value Bleed stepper 24 V (GX12-2) -> Bleed stepper signals (GX16-8); footprint Connector_Phoenix_MSTB:PhoenixContact_MSTBA_2,5_2-G-5,08_1x02_P5.08mm_Horizontal -> Connector_Phoenix_MC:PhoenixContact_MC_1,5_8-G-3.81_1x08_P3.81mm_Horizontal; symbol FlowBench:Conn_01x02 -> FlowBench:Conn_01x08
- J20: value Lift stepper signals (GX16-8) -> Bleed stepper 24 V (GX12-2); footprint Connector_Phoenix_MC:PhoenixContact_MC_1,5_8-G-3.81_1x08_P3.81mm_Horizontal -> Connector_Phoenix_MSTB:PhoenixContact_MSTBA_2,5_2-G-5,08_1x02_P5.08mm_Horizontal; symbol FlowBench:Conn_01x08 -> FlowBench:Conn_01x02
- J21: value Lift stepper 24 V (GX12-2) -> Lift stepper signals (GX16-8); footprint Connector_Phoenix_MSTB:PhoenixContact_MSTBA_2,5_2-G-5,08_1x02_P5.08mm_Horizontal -> Connector_Phoenix_MC:PhoenixContact_MC_1,5_8-G-3.81_1x08_P3.81mm_Horizontal; symbol FlowBench:Conn_01x02 -> FlowBench:Conn_01x08
- J22: value Motor housing coils (GX16-8) -> Lift stepper 24 V (GX12-2); footprint Connector_Phoenix_MC:PhoenixContact_MC_1,5_8-G-3.81_1x08_P3.81mm_Horizontal -> Connector_Phoenix_MSTB:PhoenixContact_MSTBA_2,5_2-G-5,08_1x02_P5.08mm_Horizontal; symbol FlowBench:Conn_01x08 -> FlowBench:Conn_01x02
- J23: value Motors-armed lamp -> Motor housing coils (GX16-8); footprint Connector_Phoenix_MC:PhoenixContact_MC_1,5_2-G-3.81_1x02_P3.81mm_Horizontal -> Connector_Phoenix_MC:PhoenixContact_MC_1,5_8-G-3.81_1x08_P3.81mm_Horizontal; symbol FlowBench:Conn_01x02 -> FlowBench:Conn_01x08
- J24: value E-stop (2 NC contacts) -> Motors-armed lamp; footprint Connector_Phoenix_MC:PhoenixContact_MC_1,5_4-G-3.81_1x04_P3.81mm_Horizontal -> Connector_Phoenix_MC:PhoenixContact_MC_1,5_2-G-3.81_1x02_P3.81mm_Horizontal; symbol FlowBench:Conn_01x04 -> FlowBench:Conn_01x02
- R103, R104, R105, R106, R107, R108, R109: value 4.7k -> 10k
- R110: value 470R -> 10k
- R111: value 470R -> 4.7k
- R112: value 220k -> 4.7k
- R113: value 1.5k -> 4.7k
- R114, R115, R116, R117: value 10k -> 4.7k
- R118, R119: value 10k -> 470R
- R120: value 10k -> 220k
Connections:
- net +24V_FIELD: now also J25.3 (Pin_3); no longer J24.3 (Pin_3)
- net +3V3: now also J18.9 (Pin_9), R103.1, R104.1, R105.1, R106.1, R107.1, R108.1, R109.1, R110.1, R88.1, PROTO1.1 (+3V3 rail); no longer R92.1, R93.1, R94.1, R95.1, R96.1, R97.1, R98.1, R99.1
- net +5V: now also R118.1, R119.1, R120.1, PROTO1.2 (+5V rail); no longer R110.1, R111.1, R112.1
- net BLEED_24V_F: now also J20.1 (Pin_1); no longer J19.1 (Pin_1)
- net BLEED_ALM_N: now also R108.2; no longer R100.2
- net BLEED_ALM_P: now also J19.7 (Pin_7); no longer J18.7 (Pin_7)
- net BLEED_ALM_R: now also R118.2; no longer R110.2
- net BLEED_DIR_N: now also J19.4 (Pin_4); no longer J18.4 (Pin_4)
- net BLEED_DIR_P: now also J19.3 (Pin_3); no longer J18.3 (Pin_3)
- net BLEED_ENA: now also R98.1; no longer R90.1
- net BLEED_ENA_N: now also J19.6 (Pin_6); no longer J18.6 (Pin_6)
- net BLEED_ENA_P: now also J19.5 (Pin_5); no longer J18.5 (Pin_5)
- net BLEED_HOME_IN: now also R112.1; no longer R104.1
- net BLEED_HOME_IN_R: now also R112.2; no longer R104.2
- net BLEED_HOME_N: now also R101.2; no longer R93.2
- net BLEED_PUL_N: now also J19.2 (Pin_2); no longer J18.2 (Pin_2)
- net BLEED_PUL_P: now also J19.1 (Pin_1); no longer J18.1 (Pin_1)
- net BLEED_PWR_EN: now also R96.1; no longer R88.1
- net COIL1_CMD: now also R89.1
- net COIL1_RET: now also J23.2 (Pin_2); no longer J22.2 (Pin_2)
- net COIL2_CMD: now also R90.1
- net COIL2_RET: now also J23.3 (Pin_3); no longer J22.3 (Pin_3)
- net COIL3_CMD: now also R91.1
- net COIL3_RET: now also J23.4 (Pin_4); no longer J22.4 (Pin_4)
- net COIL4_CMD: now also R92.1
- net COIL4_RET: now also J23.5 (Pin_5); no longer J22.5 (Pin_5)
- net COIL5_CMD: now also R93.1
- net COIL5_RET: now also J23.6 (Pin_6); no longer J22.6 (Pin_6)
- net COIL6_CMD: now also R94.1
- net COIL6_RET: now also J23.7 (Pin_7); no longer J22.7 (Pin_7)
- net COIL_24V: now also J25.1 (Pin_1); no longer J24.1 (Pin_1)
- net COIL_24V_ESTOP: now also J24.1 (Pin_1), J25.2 (Pin_2), R122.1, R123.1, R124.1, R125.1, R126.1, R127.1, R128.1; no longer J22.1 (Pin_1), J24.2 (Pin_2), R114.1, R115.1, R116.1, R117.1, R118.1, R119.1, R120.1
- net EFUSE_FLT_N: now also R109.2; no longer R101.2
- net ESTOP_OK_N: now also R100.2; no longer R92.2
- net ESTOP_STAT_IN: now also R111.1, J25.4 (Pin_4); no longer J24.4 (Pin_4), R103.1
- net ESTOP_STAT_IN_R: now also R111.2; no longer R103.2
- net ETH_INT_EXP: now also R110.2; no longer R102.2
- net EXP_INT_N: now also R88.2
- net GND: now also J18.10 (Pin_10), J19.8 (Pin_8), J20.2 (Pin_2), J21.8 (Pin_8), J22.2 (Pin_2), R92.2, R93.2, R94.2, R95.2, R96.2, R97.2, R98.2, R99.2, PROTO1.3 (GND rail); no longer J18.8 (Pin_8), J19.2 (Pin_2), J20.8 (Pin_8), J21.2 (Pin_2), R88.2
- net LAMP_CMD: now also R95.1
- net LAMP_RET: now also J24.2 (Pin_2); no longer J23.2 (Pin_2)
- net LED_ARMED_A: now also R122.2; no longer R114.2
- net LED_K1_A: now also R123.2; no longer R115.2
- net LED_K2_A: now also R124.2; no longer R116.2
- net LED_K3_A: now also R125.2; no longer R117.2
- net LED_K4_A: now also R126.2; no longer R118.2
- net LED_K5_A: now also R127.2; no longer R119.2
- net LED_K6_A: now also R128.2; no longer R120.2
- net LED_WD_A: now also R121.2; no longer R113.2
- net LIFT_24V_F: now also J22.1 (Pin_1); no longer J21.1 (Pin_1)
- net LIFT_ALM_N: now also R105.2; no longer R97.2
- net LIFT_ALM_P: now also J21.7 (Pin_7); no longer J20.7 (Pin_7)
- net LIFT_ALM_R: now also R119.2; no longer R111.2
- net LIFT_DIR_N: now also J21.4 (Pin_4); no longer J20.4 (Pin_4)
- net LIFT_DIR_P: now also J21.3 (Pin_3); no longer J20.3 (Pin_3)
- net LIFT_ENA: now also R99.1; no longer R91.1
- net LIFT_ENA_N: now also J21.6 (Pin_6); no longer J20.6 (Pin_6)
- net LIFT_ENA_P: now also J21.5 (Pin_5); no longer J20.5 (Pin_5)
- net LIFT_HOME_IN: now also R113.1; no longer R105.1
- net LIFT_HOME_IN_R: now also R113.2; no longer R105.2
- net LIFT_HOME_N: now also R106.2; no longer R98.2
- net LIFT_MAX_IN: now also R114.1; no longer R106.1
- net LIFT_MAX_IN_R: now also R114.2; no longer R106.2
- net LIFT_MAX_N: now also R107.2; no longer R99.2
- net LIFT_PUL_N: now also J21.2 (Pin_2); no longer J20.2 (Pin_2)
- net LIFT_PUL_P: now also J21.1 (Pin_1); no longer J20.1 (Pin_1)
- net LIFT_PWR_EN: now also R97.1; no longer R89.1
- net ORIF_B0_IN: now also R115.1; no longer R107.1
- net ORIF_B0_IN_R: now also R115.2; no longer R107.2
- net ORIF_B0_N: now also R102.2; no longer R94.2
- net ORIF_B1_IN: now also R116.1; no longer R108.1
- net ORIF_B1_IN_R: now also R116.2; no longer R108.2
- net ORIF_B1_N: now also R103.2; no longer R95.2
- net ORIF_B2_IN: now also R117.1; no longer R109.1
- net ORIF_B2_IN_R: now also R117.2; no longer R109.2
- net ORIF_B2_N: now also R104.2; no longer R96.2
- net WD_OK: now also R121.1; no longer R113.1
- net WD_RC: now also R120.2; no longer R112.2
- new net MUX4_SCL: J18.2 (Pin_2)
- new net MUX4_SDA: J18.1 (Pin_1)
- new net MUX5_SCL: J18.4 (Pin_4)
- new net MUX5_SDA: J18.3 (Pin_3)
- new net MUX6_SCL: J18.6 (Pin_6)
- new net MUX6_SDA: J18.5 (Pin_5)
- new net MUX7_SCL: J18.8 (Pin_8)
- new net MUX7_SDA: J18.7 (Pin_7)
Other:
- note added: "Prototyping area: 10 x 7 plated holes (+3V3 row, +5V row, 4 free rows, GND row); spare expander and I2C ch4-7 headers beside it. No 24 V."
- moved on the sheet: C36, C37, C38, C39, C40, C41, J17, LED10, LED11, LED12, LED13, LED14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
