File: hardware/kicad/flowbench-main/network.kicad_sch (KiCad schematic)
At the start: 22 parts, among them J4 microSD push-push, U3 WIZ850io

Commit message: KiCad: 180 x 125 mm layout, status LEDs, grouped test-point areas
- Board shrinks from 220 x 160 to 180 x 125 mm with connectors on all four
  edges; 1.0 mm between parts kept for hand soldering.
- 24 status LEDs: power rails, eFuse fault, stepper alarms, watchdog, armed,
  stepper power, each contactor coil, and every switch input (in series with
  its opto, no extra resistor).
- Scattered test points replaced by grouped areas: 24 V loops, logic-supply
  loops, and controller, analog and Digimatic 2-row headers with a GND row.
  No test points on SPI/SD lines.
- LED, test point and test header labels stay on the silkscreen.

Co-Authored-By: Claude Opus 5.5 <noreply@anthropic.com>
Claude-Session: https://claude.ai/code/session_01QEmmugJA9S77dSDSNcKrPa
Parts:
- removed J4: microSD push-push, Connector_Card:microSD_HC_Hirose_DM3AT-SF-PEJM5, symbol FlowBench:Micro_SD_Card_Det
- removed R16, R17, R18, R19, R20, R21, R22: 10k, Resistor_SMD:R_0805_2012Metric, symbol FlowBench:R
- removed TP13: SPI_SCK, TestPoint:TestPoint_Loop_D2.50mm_Drill1.0mm, symbol FlowBench:TestPoint
- removed TP14: SD_CLK, TestPoint:TestPoint_Loop_D2.50mm_Drill1.0mm, symbol FlowBench:TestPoint
- removed TP15: SD_CMD, TestPoint:TestPoint_Loop_D2.50mm_Drill1.0mm, symbol FlowBench:TestPoint
- removed TP16: SD_DAT0, TestPoint:TestPoint_Loop_D2.50mm_Drill1.0mm, symbol FlowBench:TestPoint
- added J5: microSD push-push, Connector_Card:microSD_HC_Hirose_DM3AT-SF-PEJM5, symbol FlowBench:Micro_SD_Card_Det
- added R26, R27, R28, R29, R30, R31: 10k, Resistor_SMD:R_0805_2012Metric, symbol FlowBench:R
- added R32: 33R, Resistor_SMD:R_0805_2012Metric, symbol FlowBench:R
- R25: value 33R -> 10k
Connections:
- net +3V3: now also R25.1, J5.4 (VDD), R26.1, R27.1, R28.1, R29.1, R30.1, R31.1
- net ETH_CS: now also R23.2
- net ETH_INT_N: now also R24.2
- net ETH_RST_N: now also R25.2
- net GND: now also J5.6 (VSS), J5.9 (DET_B), J5.SH (SHIELD)
- net SD_CD_N: now also J5.10 (DET_A), R31.2; no longer R24.2
- net SD_CLK: now also J5.5 (CLK), R32.2; no longer R25.2
- net SD_CLK_MCU: now also R32.1; no longer R25.1
- net SD_CMD: now also J5.3 (CMD), R26.2
- net SD_DAT0: now also J5.7 (DAT0), R27.2
- net SD_DAT1: now also J5.8 (DAT1), R28.2
- net SD_DAT2: now also J5.1 (DAT2), R29.2
- net SD_DAT3: now also J5.2 (DAT3/CD), R30.2; no longer R23.2
Other:
- note added: "Fast lines (SPI, SD) have no test points: probe them at the WIZ850io and microSD pins."
- moved on the sheet: C6, C7, C8, C9, JP1, JP2, R23, R24, R25, U3
