File: hardware/kicad/flowbench-main/power.kicad_sch (KiCad schematic)
At the start: 42 parts, among them J1 24V IN, J2 PM1 power socket, J3 PM1 signal socket, Q1 SUD50P06-15 (60 V P-ch, DPAK), Q2 MMBT3904, Q3 SUD50P06-15 (60 V P-ch, DPAK), Q4 MMBT3904, Q5 SUD50P06-15 (60 V P-ch, DPAK), Q6 MMBT3904, U1 LM1117-3.3

Commit message: KiCad: 180 x 125 mm layout, status LEDs, grouped test-point areas
- Board shrinks from 220 x 160 to 180 x 125 mm with connectors on all four
  edges; 1.0 mm between parts kept for hand soldering.
- 24 status LEDs: power rails, eFuse fault, stepper alarms, watchdog, armed,
  stepper power, each contactor coil, and every switch input (in series with
  its opto, no extra resistor).
- Scattered test points replaced by grouped areas: 24 V loops, logic-supply
  loops, and controller, analog and Digimatic 2-row headers with a GND row.
  No test points on SPI/SD lines.
- LED, test point and test header labels stay on the silkscreen.

Co-Authored-By: Claude Opus 5.5 <noreply@anthropic.com>
Claude-Session: https://claude.ai/code/session_01QEmmugJA9S77dSDSNcKrPa
Parts:
- added LED1: +24V, LED_SMD:LED_0805_2012Metric, symbol FlowBench:LED
- added LED2: +12V, LED_SMD:LED_0805_2012Metric, symbol FlowBench:LED
- added LED3: +5V, LED_SMD:LED_0805_2012Metric, symbol FlowBench:LED
- added LED4: +3V3, LED_SMD:LED_0805_2012Metric, symbol FlowBench:LED
- added LED5: EFUSE FLT, LED_SMD:LED_0805_2012Metric, symbol FlowBench:LED
- added LED6: BLEED PWR, LED_SMD:LED_0805_2012Metric, symbol FlowBench:LED
- added LED7: LIFT PWR, LED_SMD:LED_0805_2012Metric, symbol FlowBench:LED
- added R13, R18, R19: 10k, Resistor_SMD:R_0805_2012Metric, symbol FlowBench:R
- added R14: 4.7k, Resistor_SMD:R_0805_2012Metric, symbol FlowBench:R
- added R15: 1.5k, Resistor_SMD:R_0805_2012Metric, symbol FlowBench:R
- added R16: 680R, Resistor_SMD:R_0805_2012Metric, symbol FlowBench:R
- added R17: 1k, Resistor_SMD:R_0805_2012Metric, symbol FlowBench:R
- added TP10: +5VA, TestPoint:TestPoint_Loop_D2.50mm_Drill1.0mm, symbol FlowBench:TestPoint
- added TP11: +3V3, TestPoint:TestPoint_Loop_D2.50mm_Drill1.0mm, symbol FlowBench:TestPoint
- added TP12, TP7: GND, TestPoint:TestPoint_Loop_D2.50mm_Drill1.0mm, symbol FlowBench:TestPoint
- added TP8: +12V, TestPoint:TestPoint_Loop_D2.50mm_Drill1.0mm, symbol FlowBench:TestPoint
- added TP9: +5V, TestPoint:TestPoint_Loop_D2.50mm_Drill1.0mm, symbol FlowBench:TestPoint
- TP1: value +24V -> +24V_RAW
- TP2: value +12V -> +24V
- TP3: value +5V -> BLEED_24V_F
- TP4: value +3V3 -> LIFT_24V_F
- TP5: value +5VA -> COIL_24V_ESTOP
- TP6: value GND -> +24V_FIELD
Connections:
- net +12V: now also R14.1, TP8.1; no longer TP2.1
- net +24V: now also TP2.1, R13.1; no longer TP1.1
- net +24V_FIELD: now also TP6.1
- net +24V_RAW: now also TP1.1
- net +3V3: now also R16.1, R17.1, TP11.1; no longer TP4.1
- net +5V: now also R15.1, TP9.1; no longer TP3.1
- net +5VA: now also TP10.1; no longer TP5.1
- net BLEED_24V_F: now also TP3.1, R18.1
- net EFUSE_FLT_N: now also LED5.1 (K)
- net GND: now also LED1.1 (K), LED2.1 (K), LED3.1 (K), LED4.1 (K), LED6.1 (K), LED7.1 (K), TP12.1, TP7.1; no longer TP6.1
- net LIFT_24V_F: now also TP4.1, R19.1
- new net COIL_24V_ESTOP: TP5.1
- new net LED_12V_A: LED2.2 (A), R14.2
- new net LED_24V_A: LED1.2 (A), R13.2
- new net LED_3V3_A: LED4.2 (A), R16.2
- new net LED_5V_A: LED3.2 (A), R15.2
- new net LED_BLEEDPWR_A: LED6.2 (A), R18.2
- new net LED_FLT_A: LED5.2 (A), R17.2
- new net LED_LIFTPWR_A: LED7.2 (A), R19.2
Other:
- note added: "Test points: 24 V area (supply, stepper and coil feeds) kept apart from the logic-supply area."
- moved on the sheet: C1, C2, C3, C4, C5, F1, F2, F3, H1, H2, H3, H4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
