File: hardware/kicad/flowbench-main/sensors.kicad_sch (KiCad schematic)
At the start: 37 parts, among them J5 BME280 (GX12-4), U4 TCA9548APWR, U5 ABP2DRRN100MD2A3XX, U6 ABP2DRRN100MD2A3XX, U7 ABP2DRRN100MD2A3XX, U8 ADS1219 #1 (0x40), U9 ADS1219 #2 (0x41)

Commit message: KiCad: 180 x 125 mm layout, status LEDs, grouped test-point areas
- Board shrinks from 220 x 160 to 180 x 125 mm with connectors on all four
  edges; 1.0 mm between parts kept for hand soldering.
- 24 status LEDs: power rails, eFuse fault, stepper alarms, watchdog, armed,
  stepper power, each contactor coil, and every switch input (in series with
  its opto, no extra resistor).
- Scattered test points replaced by grouped areas: 24 V loops, logic-supply
  loops, and controller, analog and Digimatic 2-row headers with a GND row.
  No test points on SPI/SD lines.
- LED, test point and test header labels stay on the silkscreen.

Co-Authored-By: Claude Opus 5.5 <noreply@anthropic.com>
Claude-Session: https://claude.ai/code/session_01QEmmugJA9S77dSDSNcKrPa
Parts:
- removed J5: BME280 (GX12-4), Connector_Phoenix_MC:PhoenixContact_MC_1,5_4-G-3.81_1x04_P3.81mm_Horizontal, symbol FlowBench:Conn_01x04
- removed R26, R27: 2.2k, Resistor_SMD:R_0805_2012Metric, symbol FlowBench:R
- removed R28: 10k, Resistor_SMD:R_0805_2012Metric, symbol FlowBench:R
- removed R29, R30, R31, R32: 4.7k, Resistor_SMD:R_0805_2012Metric, symbol FlowBench:R
- removed TP17: ADC2_AIN2, TestPoint:TestPoint_Loop_D2.50mm_Drill1.0mm, symbol FlowBench:TestPoint
- removed TP18: ADC2_AIN3, TestPoint:TestPoint_Loop_D2.50mm_Drill1.0mm, symbol FlowBench:TestPoint
- added J6: BME280 (GX12-4), Connector_Phoenix_MC:PhoenixContact_MC_1,5_4-G-3.81_1x04_P3.81mm_Horizontal, symbol FlowBench:Conn_01x04
- added J7: Analog test header, Connector_PinHeader_2.54mm:PinHeader_2x05_P2.54mm_Vertical, symbol FlowBench:Conn_02x05_Odd_Even
- added R42, R43: 4.7k, Resistor_SMD:R_0805_2012Metric, symbol FlowBench:R
- added R44, R46, R48: 10k, Resistor_SMD:R_0805_2012Metric, symbol FlowBench:R
- added R45: 150k, Resistor_SMD:R_0805_2012Metric, symbol FlowBench:R
- added R47: 30k, Resistor_SMD:R_0805_2012Metric, symbol FlowBench:R
- R33, R34: value 4.7k -> 2.2k
- R35: value 4.7k -> 10k
- R37, R39, R41: value 10k -> 4.7k
- R38: value 150k -> 4.7k
- R40: value 30k -> 4.7k
Connections:
- net +24V: now also R45.1; no longer R38.1
- net +3V3: now also R38.1, R39.1, R40.1, R41.1, J6.1 (Pin_1), R42.1, R43.1, R44.1
- net +5VA: now also R47.1; no longer R40.1
- net ADC2_AIN2: now also J7.1 (Pin_1)
- net ADC2_AIN3: now also J7.3 (Pin_3)
- net ADC_RST_N: now also R44.2; no longer R37.2
- net GND: now also J6.2 (Pin_2), J7.10 (Pin_10), J7.2 (Pin_2), J7.4 (Pin_4), J7.6 (Pin_6), J7.8 (Pin_8), R46.2, R48.2; no longer R39.2, R41.2
- net MAF_ID_ADC: now also J7.7 (Pin_7)
- net MAF_SIG_ADC: now also J7.5 (Pin_5)
- net MON_24V: now also R45.2, R46.1; no longer R38.2, R39.1
- net MON_5VA: now also R47.2, R48.1; no longer R40.2, R41.1
- net MUX0_SCL: now also R37.2
- net MUX0_SDA: now also R36.2
- net MUX1_SCL: now also R39.2
- net MUX1_SDA: now also R38.2
- net MUX2_SCL: now also R41.2; no longer R34.2
- net MUX2_SDA: now also R40.2; no longer R33.2
- net MUX3_SCL: now also J6.4 (Pin_4), R43.2; no longer R36.2
- net MUX3_SDA: now also J6.3 (Pin_3), R42.2; no longer R35.2
- net MUX_RST_N: now also R35.2
- net SCL: now also R34.2
- net SDA: now also R33.2
- new net CT_BIAS: J7.9 (Pin_9)
Other:
- note added: "Analog test header (2x5): ADC2 spare inputs AIN2/AIN3, MAF signal and harness ID at the ADC, current-sensor bias."
- moved on the sheet: C10, C11, C12, C13, C14, C15, C16, C17, C18, C19, C20, C21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

Commit message: KiCad: prototyping area with I2C expansion header
- 10 x 7 plated-hole grid (+3V3 row, +5V row, 4 free rows, GND row) between
  the optocouplers and the multiplexer; footprint FlowBench:ProtoArea_10x7.
- Multiplexer channels 4-7 now brought out with 4.7k pull-ups to a new I2C
  expansion header beside the grid; the expander 2 spare header moves there too.
- ATtiny, 74LVC14 and Digimatic test header nudged to keep 1 mm clearance.

Co-Authored-By: Claude Opus 5.5 <noreply@anthropic.com>
Claude-Session: https://claude.ai/code/session_01QEmmugJA9S77dSDSNcKrPa
Parts:
- added R49, R50, R51: 4.7k, Resistor_SMD:R_0805_2012Metric, symbol FlowBench:R
- added R52, R54, R56: 10k, Resistor_SMD:R_0805_2012Metric, symbol FlowBench:R
- added R53: 150k, Resistor_SMD:R_0805_2012Metric, symbol FlowBench:R
- added R55: 30k, Resistor_SMD:R_0805_2012Metric, symbol FlowBench:R
- R44, R46, R48: value 10k -> 4.7k
- R45: value 150k -> 4.7k
- R47: value 30k -> 4.7k
Connections:
- net +24V: now also R53.1; no longer R45.1
- net +3V3: now also R45.1, R46.1, R47.1, R48.1, R49.1, R50.1, R51.1, R52.1
- net +5VA: now also R55.1; no longer R47.1
- net ADC_RST_N: now also R52.2; no longer R44.2
- net GND: now also R54.2, R56.2; no longer R46.2, R48.2
- net MON_24V: now also R53.2, R54.1; no longer R45.2, R46.1
- net MON_5VA: now also R55.2, R56.1; no longer R47.2, R48.1
- net MUX4_SDA: now reaches U4.13 (SD4)
- net MUX4_SDA: now also R44.2
- net MUX4_SCL: now reaches U4.14 (SC4)
- net MUX4_SCL: now also R45.2
- net MUX5_SDA: now reaches U4.15 (SD5)
- net MUX5_SDA: now also R46.2
- net MUX5_SCL: now reaches U4.16 (SC5)
- net MUX5_SCL: now also R47.2
- net MUX6_SDA: now reaches U4.17 (SD6)
- net MUX6_SDA: now also R48.2
- net MUX6_SCL: now reaches U4.18 (SC6)
- net MUX6_SCL: now also R49.2
- net MUX7_SDA: now reaches U4.19 (SD7)
- net MUX7_SDA: now also R50.2
- net MUX7_SCL: now reaches U4.20 (SC7)
- net MUX7_SCL: now also R51.2
- no-connect marks 16 -> 8
Other:
- note added: "Behind the mux: ABP2 reference ch0, orifice ch1, pitot ch2 (all 0x28), BME280 cable ch3 (0x77). Ch4-7 go to the prototyping area."
- note removed: "Behind the mux: ABP2 reference ch0, orifice ch1, pitot ch2 (all 0x28), BME280 cable ch3 (0x77). Ch4-7 spare."
- moved on the sheet: C11, C12, C13, C14, C15, C16, C17, C18, C19, C20, C21, J6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
